File: stm32-led-strip-controller.kicad_pcb (KiCad board)
At the start: 4 copper layers, 71 x 54 mm, 62 parts, among them J101 Tag Connector, J102 Barrel_Jack_Switch, J104 JST 2.54 Header, J106 JST 2.54 Header, SW101 SW_DIP_x04, SW106 SW_Push, U101 STM32F401RCTx, U102 USBLC6-2SC6, U103 74AHCT1G125, U104 M24C64-RMN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

Commit message: update pcb
Parts:
- removed H101, H103: MountingHole, MountingHole:MountingHole_3.2mm_M3_Pad_Via
- removed RN101: 10K, Resistor_SMD:R_Array_Convex_4x0603
- removed SW101: SW_DIP_x04, User_Footprint:SMDIP-8_W6.6mm
- J102: footprint Connector_BarrelJack:BarrelJack_Wuerth_6941xx301002 -> User_Footprint:BarrelJack_GCT_DCJ250-10-A-K1-K; moved to B.Cu
- J104: footprint Connector_JST:JST_XH_B3B-XH-A_1x03_P2.50mm_Vertical -> Connector_JST:JST_XH_S3B-XH-A-1_1x03_P2.50mm_Horizontal; moved to B.Cu
- J106, OLED101: moved to B.Cu
- moved L301 76.9 mm to (84.5, 70.7), turned to -90 degrees
- moved C305 71.2 mm to (86.5, 78.0), turned to -90 degrees
- moved C304 67.0 mm to (89.5, 71.0), turned to 90 degrees
- moved C303 66.1 mm to (91.5, 71.0), turned to 90 degrees
- moved C301 64.8 mm to (89.1, 63.7)
- moved C302 64.4 mm to (89.1, 65.2)
- moved R301 64.3 mm to (86.8, 62.9), turned to 90 degrees
- moved U301 63.9 mm to (90.4, 67.2)
- moved R303 62.8 mm to (86.8, 59.8), turned to 90 degrees
- moved R302 59.8 mm to (93.3, 70.9), turned to 90 degrees
- moved R304 57.8 mm to (92.3, 65.2), turned to 180 degrees
- moved J102 56.7 mm to (79.3, 63.4), turned to 0 degrees
- moved J104 56.5 mm to (135.2, 61.5)
- moved U103 56.2 mm to (140.2, 63.6)
- moved C118 53.5 mm to (139.7, 67.3), turned to -90 degrees
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Connections:
- C303 pad 1: /BUCK_5V/VOUT -> +5V
- C304 pad 1: /BUCK_5V/VOUT -> +5V
- C305 pad 1: /BUCK_5V/VOUT -> +5V
- D103 pad 2: +5V -> Net-(D103-A)
- F101 pad 1: /BUCK_5V/VOUT -> +5V
- F101 pad 2: +5V -> Net-(D103-A)
- L301 pad 2: /BUCK_5V/VOUT -> +5V
- R302 pad 1: /BUCK_5V/VOUT -> +5V
Routing:
- net +5V: track 20.0 -> 60.9 mm
- net /SCL: track 25.6 -> 52.2 mm
- net /SDA: track 25.7 -> 50.9 mm, vias 3 -> 4
- net /~{OE}: track 27.9 -> 52.2 mm, vias 0 -> 2
- net /DIP3: track 17.7 -> 0.00 mm
- net Net-(U301-EN): track 0.00 -> 16.7 mm, vias 0 -> 2
- net /DIP2: track 16.1 -> 0.00 mm
- net /RGB_LED: track 30.5 -> 45.2 mm
- net /DIP1: track 14.4 -> 0.00 mm
- net /BOOT0: track 11.5 -> 0.00 mm
- net Net-(U301-FB): track 0.00 -> 9.92 mm
- net GND: track 97.8 -> 106.1 mm, vias 31 -> 39
- net VBUS: track 6.34 -> 1.53 mm, vias 4 -> 0
- net /IR_RECV: track 33.0 -> 37.5 mm
- net Net-(R104-Pad2): track 6.17 -> 1.80 mm
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- added copper zone on F.Cu, net Net-(U301-SW)
- removed copper zone on B.Cu, net VBUS
Other:
- board size 71 x 54 mm -> 75 x 38 mm
- board text added: "${TITLE} Rev. ${REVISION} / ${ISSUE_DATE}"
- board text added: "12V/5A DC Power"
- board text removed: "+"
- board text removed: "-"
- board text removed: "CR1220"
- board text removed: "Clock"
- board text removed: "Status"
- board text removed: "locked"
